File: hardware/turbocan.kicad_pcb (KiCad board)
At the start: 2 copper layers, 43 x 43 mm, 88 parts, among them J1 USB_C_Receptacle_USB2.0, J10 CAN_PORT, J11 FAN0, J12 FAN1, J13 HEAT, J14 PROBE, J2 STEPPER, J5 DEBUG, J7 ENDSTOPX, J8 ENDSTOPY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

Commit message: Total reroute, move to 4 layer board, change mcu to more available stm32f103
Parts:
- removed D4: BAT42W, Diode_SMD:D_SOD-123
- U8: value STM32F072CBUx -> STM32F103C8Tx; footprint Package_DFN_QFN:QFN-48-1EP_7x7mm_P0.5mm_EP5.6x5.6mm -> Package_QFP:LQFP-48_7x7mm_P0.5mm
- moved C17 19.1 mm to (51.0, 25.9), turned to 0 degrees
- moved R16 10.0 mm to (53.6, 47.6), turned to 0 degrees
- moved J2 7.60 mm to (47.0, 45.2), turned to 90 degrees
- moved R14 7.13 mm to (51.0, 27.4), turned to 0 degrees
- moved C13 4.88 mm to (31.3, 34.7)
- moved C15 4.88 mm to (35.7, 34.7)
- moved C14 4.88 mm to (33.5, 34.7)
- moved C23 4.35 mm to (31.9, 29.4)
- moved R15 3.94 mm to (50.6, 40.5)
- moved L2 3.88 mm to (32.8, 31.8)
- moved R19 3.83 mm to (47.1, 47.9)
- moved C7 3.42 mm to (34.6, 45.5)
- moved R25 3.32 mm to (37.9, 45.5)
- moved R20 3.13 mm to (32.0, 26.9), turned to 0 degrees
- moved C19 2.61 mm to (31.9, 28.4)
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Connections:
- J1 pad A8: (no net) -> unconnected-(J1-PadA8)
- J1 pad B8: (no net) -> unconnected-(J1-PadB8)
- J14 pad 1: +24V -> +5V
- J14 pad 3: Net-(D4-Pad1) -> Net-(C20-Pad1)
- U3 pad 5: (no net) -> unconnected-(U3-Pad5)
- U8 pad 11: LED -> ENDSTOPX
- U8 pad 13: FAN1 -> ENDSTOPY
- U8 pad 18: (no net) -> unconnected-(U8-Pad18)
- U8 pad 2: (no net) -> LED
- U8 pad 21: (no net) -> FAN1
- U8 pad 3: (no net) -> unconnected-(U8-Pad3)
- U8 pad 38: (no net) -> unconnected-(U8-Pad38)
- U8 pad 39: (no net) -> unconnected-(U8-Pad39)
- U8 pad 4: (no net) -> unconnected-(U8-Pad4)
- U8 pad 42: ENDSTOPX -> unconnected-(U8-Pad42)
- U8 pad 43: ENDSTOPY -> unconnected-(U8-Pad43)
- U9 pad 10: (no net) -> unconnected-(U9-Pad10)
- U9 pad 11: (no net) -> unconnected-(U9-Pad11)
- U9 pad 3: (no net) -> unconnected-(U9-Pad3)
- U9 pad 8: (no net) -> unconnected-(U9-Pad8)
- U9 pad 9: (no net) -> unconnected-(U9-Pad9)
Routing:
- net +3V3: track 163.8 -> 18.6 mm
- net GND: track 31.8 -> 7.30 mm, vias 78 -> 13
- net FAN1: track 31.2 -> 15.0 mm, vias 2 -> 0
- net INDEX: track 44.6 -> 28.9 mm, vias 3 -> 1
- net ENDSTOPY: track 33.4 -> 21.0 mm, vias 2 -> 0
- net DIAG: track 46.6 -> 35.7 mm, vias 2 -> 1
- net BOOT0: track 28.9 -> 18.2 mm, vias 0 -> 1
- net Net-(J2-Pad1): track 17.5 -> 7.06 mm
- net /SWITCH: track 0.00 -> 10.1 mm
- net NRST: track 31.4 -> 21.4 mm, vias 3 -> 1
- net TH0: track 28.6 -> 38.6 mm, vias 0 -> 1
- net Net-(J13-Pad1): track 9.63 -> 0.00 mm
- net ENDSTOPX: track 23.1 -> 15.2 mm, vias 2 -> 0
- net CANL: track 28.8 -> 22.1 mm, vias 0 -> 1
- net +5V: track 66.1 -> 72.4 mm, vias 5 -> 4
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- added copper zone on In2.Cu, net +3V3
- added copper zone on In1.Cu, net GND
- added copper zone on F.Cu, net Net-(J13-Pad1)
Other:
- board size 43 x 43 mm -> 43.3 x 43 mm
- copper layers 2 -> 4
- net class 0.5mm removed
- net class 1mm removed
- net class Default removed
- board text added: "TurboCAN v0.3.1"
- board text removed: "24V"
- board text removed: "TurboCAN v0.2"
